Commit message: fixed lidar

File: src/description/urdf/robot_base.xacro (robot description, xacro)
@@ -45,5 +45,13 @@
   </gazebo>
   <link name="imu_link">
-    <origin xyz="0 0 0.15" rpy="0 0 0"/>
+    <visual>
+      <geometry>
+        <box size="0.03 0.03 0.02"/>
+      </geometry>
+      <material name="orange">
+        <color rgba="1 0.5 0 1"/>
+      </material>
+      <origin xyz="0 0 0.15" rpy="0 0 0"/>
+    </visual>
   </link>
   <joint name="imu_joint" type="fixed">
@@ -53,18 +61,34 @@
   </joint>
   <link name="gps_link">
-    <origin xyz="0 0 0.1" rpy="0 0 0"/>
+    <visual>
+      <geometry>
+        <box size="0.03 0.03 0.02"/>
+      </geometry>
+      <material name="white">
+        <color rgba="1 1 1 1"/>
+      </material>
+      <origin xyz="0 0 0.2" rpy="0 0 0"/>
+    </visual>
   </link>
   <joint name="gps_joint" type="fixed">
     <parent link="base_link"/>
     <child link="gps_link"/>
-    <origin xyz="0 0 0.1"/>
+    <origin xyz="0 0 0.2"/>
   </joint>
   <link name="lidar_link">
-    <origin xyz="0.2 0 0.15" rpy="0 0 0"/>
+    <visual>
+      <geometry>
+        <cylinder radius="0.04" length="0.05"/>
+      </geometry>
+      <origin xyz="0.1 0 0.15" rpy="0 0 0"/>
+      <material name="gray">
+        <color rgba="0.6 0.6 0.6 1.0"/>
+      </material>
+    </visual>
   </link>
   <joint name="lidar_joint" type="fixed">
     <parent link="base_link"/>
     <child link="lidar_link"/>
-    <origin xyz="0.2 0 0.15"/>
+    <origin xyz="0.11 0 0.15"/>
   </joint>
   <link name="camera_link">

File: src/description/urdf/robot_sim.xacro (robot description, xacro)
@@ -3,18 +3,9 @@
   <xacro:macro name="sim">
     <gazebo>
-  <plugin filename="gz-sim-diff-drive-system"
-          name="gz::sim::systems::DiffDrive">
-    <left_joint>front_left_wheel_joint</left_joint>
-    <left_joint>rear_left_wheel_joint</left_joint>
-    <right_joint>front_right_wheel_joint</right_joint>
-    <right_joint>rear_right_wheel_joint</right_joint>
-    <wheel_separation>0.44</wheel_separation>
-    <wheel_radius>0.075</wheel_radius>
-    <topic>/cmd_vel</topic>
-    <odom_topic>/odom</odom_topic>
-    <frame_id>odom</frame_id>
-    <child_frame_id>base_footprint</child_frame_id>
-  </plugin>
-</gazebo>
+      <plugin filename="libgz_ros2_control-system.so"
+              name="gz_ros2_control::GazeboSimROS2ControlPlugin">
+        <parameters>$(find description)/config/controllers.yaml</parameters>
+      </plugin>
+    </gazebo>
   </xacro:macro>
 </robot>
